File: kicad/nanoTracer.sch (KiCad schematic (older format))
At the start: 51 parts, among them P1 6.3_AC, P2 HEATER, P3 CONN_3, P4 HT_AC, P5 NEG_AC, U1 TL072, U2 TL071, U3 MCP4921-E/P, U4 LM337T, U5 MCP3202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

Commit message: [SCH] Move BTN_UP/BTN_DN as not connected on Arduino Zero
Connections:
- wire segments 150 -> 151
- no-connect marks 16 -> 18
Changed lines of the file:
@@
 Text Label 4200 6000 0    60   ~ 0
 IA
-Text Label 10350 3150 2    60   ~ 0
-BTN_UP
-Text Label 10350 3250 2    60   ~ 0
-BTN_DN
 Text Label 7300 4550 2    60   ~ 0
 UA
@@
 	10250 4850 10250 4950
 NoConn ~ 10550 4950
-Wire Wire Line
-	9900 3250 10350 3250
-Wire Wire Line
-	10350 3150 9900 3150
 Text Label 10000 5150 0    60   ~ 0
 BTN_UP
@@
 BTN_DN
 Wire Wire Line
-	10550 5150 10000 5150
-Wire Wire Line
-	10550 5250 10000 5250
+	8000 5150 10550 5150
+Wire Wire Line
+	7900 5250 10550 5250
 $Comp
 L ARDUINO_SHIELD SHIELD1
@@
 	1    0    0    -1
 $EndComp
-NoConn ~ 8000 4850
-NoConn ~ 8000 4950
 NoConn ~ 9900 4850
 NoConn ~ 9900 4950
@@
 Wire Notes Line
 	4300 5400 6050 5400
+NoConn ~ 9900 3450
+NoConn ~ 9900 3350
+NoConn ~ 9900 3250
+NoConn ~ 9900 3150
+Wire Wire Line
+	8000 5150 8000 4950
+Wire Wire Line
+	7900 5250 7900 4850
+Wire Wire Line
+	7900 4850 8000 4850
 $EndSCHEMATC

Commit message: Switch to 10-pin header w/I2C for expansion port
Parts:
- removed U6: SIL12, Pin_Headers:Pin_Header_Straight_1x12, symbol SIL12
- added J1: SIL10, Pin_Headers:Pin_Header_Straight_1x10, symbol SIL10
Connections:
- net labels added: SCL, SDA
- net labels removed: BTN_DN, BTN_OK, BTN_UP
- wire segments 151 -> 150
Changed lines of the file:
@@
 Wire Wire Line
 	8000 4450 7550 4450
-Text Label 10300 4750 2    60   ~ 0
-BTN_OK
-Text Label 10300 4650 2    60   ~ 0
-LCD_RS
-Text Label 10300 4550 2    60   ~ 0
-LCD_EN
 Text Label 10300 4450 2    60   ~ 0
-LCD_D4
+LCD_D5
 Text Label 10300 4350 2    60   ~ 0
-LCD_D5
+LCD_D6
 Text Label 10300 4250 2    60   ~ 0
-LCD_D6
-Text Label 10300 4050 2    60   ~ 0
 LCD_D7
 Wire Wire Line
@@
 	4850 5650 4850 5700
 $Comp
-L SIL12 U6
-U 1 1 5790F8A0
-P 10900 4700
-F 0 "U6" H 10950 5350 50  0000 C CNN
-F 1 "SIL12" V 10930 4700 50  0000 C CNN
-F 2 "Pin_Headers:Pin_Header_Straight_1x12" H 10900 4700 50  0001 C CNN
-F 3 "" H 10900 4700 50  0000 C CNN
-	1    10900 4700
-	1    0    0    1
-$EndComp
-$Comp
 L GND #PWR034
 U 1 1 57910308
-P 10250 4950
-F 0 "#PWR034" H 10250 4950 30  0001 C CNN
-F 1 "GND" H 10250 4880 30  0001 C CNN
-F 2 "" H 10250 4950 60  0000 C CNN
-F 3 "" H 10250 4950 60  0000 C CNN
-	1    10250 4950
+P 10400 4900
+F 0 "#PWR034" H 10400 4900 30  0001 C CNN
+F 1 "GND" H 10400 4830 30  0001 C CNN
+F 2 "" H 10400 4900 60  0000 C CNN
+F 3 "" H 10400 4900 60  0000 C CNN
+	1    10400 4900
 	-1   0    0    -1
 $EndComp
@@
 L VDD #PWR035
 U 1 1 579103AF
-P 10400 5000
-F 0 "#PWR035" H 10400 5100 30  0001 C CNN
-F 1 "VDD" H 10400 5110 30  0000 C CNN
-F 2 "" H 10400 5000 60  0000 C CNN
-F 3 "" H 10400 5000 60  0000 C CNN
-	1    10400 5000
+P 10250 5000
+F 0 "#PWR035" H 10250 5100 30  0001 C CNN
+F 1 "VDD" H 10250 5110 30  0000 C CNN
+F 2 "" H 10250 5000 60  0000 C CNN
+F 3 "" H 10250 5000 60  0000 C CNN
+	1    10250 5000
 	-1   0    0    -1
 $EndComp
-Wire Wire Line
-	10550 5050 10400 5050
-Wire Wire Line
-	10400 5050 10400 5000
-Wire Wire Line
-	10550 4850 10250 4850
-Wire Wire Line
-	10250 4850 10250 4950
-NoConn ~ 10550 4950
-Text Label 10000 5150 0    60   ~ 0
-BTN_UP
-Text Label 10000 5250 0    60   ~ 0
-BTN_DN
-Wire Wire Line
-	8000 5150 10550 5150
-Wire Wire Line
-	7900 5250 10550 5250
+NoConn ~ 8000 4850
 $Comp
 L ARDUINO_SHIELD SHIELD1
@@
 Wire Wire Line
 	6900 4750 8000 4750
-Wire Wire Line
-	9900 4050 10400 4050
-Wire Wire Line
-	10400 4050 10400 4150
-Wire Wire Line
-	10400 4150 10550 4150
 Wire Notes Line
 	4300 5400 6050 5400
 NoConn ~ 9900 3450
 NoConn ~ 9900 3350
-NoConn ~ 9900 3250
-NoConn ~ 9900 3150
-Wire Wire Line
-	8000 5150 8000 4950
-Wire Wire Line
-	7900 5250 7900 4850
-Wire Wire Line
-	7900 4850 8000 4850
+NoConn ~ 9900 4050
+NoConn ~ 8000 4950
+$Comp
+L SIL10 J1
+U 1 1 57928D5A
+P 10900 4500
+F 0 "J1" H 10900 5100 50  0000 C CNN
+F 1 "SIL10" V 10920 4500 50  0000 C CNN
+F 2 "Pin_Headers:Pin_Header_Straight_1x10" H 10900 4500 50  0001 C CNN
+F 3 "" H 10900 4500 50  0000 C CNN
+	1    10900 4500
+	1    0    0    -1
+$EndComp
+Wire Wire Line
+	9900 3250 10400 3250
+Wire Wire Line
+	10400 3250 10400 4150
+Wire Wire Line
+	10400 4150 10550 4150
+Wire Wire Line
+	10550 4050 10500 4050
+Wire Wire Line
+	10500 4050 10500 3150
+Wire Wire Line
+	10500 3150 9900 3150
+Wire Wire Line
+	10400 4850 10400 4900
+Wire Wire Line
+	10400 4850 10550 4850
+Wire Wire Line
+	10550 4950 10500 4950
+Wire Wire Line
+	10500 4950 10500 5000
+Wire Wire Line
+	10500 5000 10250 5000
+Text Label 10300 3150 2    60   ~ 0
+SCL
+Text Label 10300 3250 2    60   ~ 0
+SDA
+Text Label 10300 4550 2    60   ~ 0
+LCD_D4
+Text Label 10300 4650 2    60   ~ 0
+LCD_EN
+Text Label 10300 4750 2    60   ~ 0
+LCD_RS
 $EndSCHEMATC

Commit message: First PCB version
Parts:
- removed C8, C9: 100n, Capacitors_ThroughHole:C_Rect_L7_W2_P5, symbol C
- removed F1, F2, F3: FUSE, Fuse_Holders_and_Fuses:Fuseholder5x20_horiz_open_Schurter_0031_8201, symbol FUSE
- removed R1: 100k, Resistors_ThroughHole:Resistor_Horizontal_RM10mm, symbol R-RESCUE-nanoTracer
- C4, C5: footprint Capacitors_ThroughHole:C_Rect_L7_W2_P5 -> Capacitors_ThroughHole:C_Rect_L18_W6_H12_P15
- R11: value R -> R11
- R2: value R -> R2
- R3: value R -> R3
- R4: value R -> R4
Connections:
- net GRID: now also R2.2, R4.2, U1.1
- net at P1.1 (P1), P2.1 (P1): now also D1.2, D1.4
- net at P1.2 (PM), P2.2 (PM): no longer D1.2
- net at P5.1 (P1): now also C5.1, D3.2, R9.2
- net at C4.1, D3.4, R8.2: now also P5.2 (PM)
- net at JP1.2: now also SHIELD1.AD3; no longer SHIELD1.AD2
- net at JP2.2: now also SHIELD1.AD2; no longer SHIELD1.AD3
- net at P4.1 (P1): now also C4.2, D2.4
Other:
- moved on the sheet: JP1, JP2, P3, R4
Changed lines of the file:
@@
 P 2600 7200
 F 0 "R11" V 2600 7200 40  0000 C CNN
-F 1 "R" V 2607 7201 40  0001 C CNN
+F 1 "R11" V 2607 7201 40  0001 C CNN
 F 2 "Resistors_ThroughHole:Resistor_Horizontal_RM10mm" V 2530 7200 30  0001 C CNN
 F 3 "~" H 2600 7200 30  0000 C CNN
@@
 L R-RESCUE-nanoTracer R4
 U 1 1 54D800CA
-P 2800 4850
-F 0 "R4" V 2800 4850 40  0000 C CNN
-F 1 "R" V 2807 4851 40  0001 C CNN
-F 2 "Resistors_ThroughHole:Resistor_Horizontal_RM10mm" V 2730 4850 30  0001 C CNN
-F 3 "~" H 2800 4850 30  0000 C CNN
-	1    2800 4850
+P 2800 4650
+F 0 "R4" V 2800 4650 40  0000 C CNN
+F 1 "R4" V 2807 4651 40  0001 C CNN
+F 2 "Resistors_ThroughHole:Resistor_Horizontal_RM10mm" V 2730 4650 30  0001 C CNN
+F 3 "~" H 2800 4650 30  0000 C CNN
+	1    2800 4650
 	0    1    -1   0
 $EndComp
-$Comp
-L R-RESCUE-nanoTracer R1
-U 1 1 54D80200
-P 1750 4050
-F 0 "R1" V 1830 4050 40  0000 C CNN
-F 1 "100k" V 1757 4051 40  0000 C CNN
-F 2 "Resistors_ThroughHole:Resistor_Horizontal_RM10mm" V 1680 4050 30  0001 C CNN
-F 3 "~" H 1750 4050 30  0000 C CNN
-	1    1750 4050
-	0    1    -1   0
-$EndComp
-Wire Wire Line
-	3150 3700 3150 4000
 $Comp
 L R-RESCUE-nanoTracer R3
@@
 P 2150 4850
 F 0 "R3" V 2150 4850 40  0000 C CNN
-F 1 "R" V 2157 4851 40  0001 C CNN
+F 1 "R3" V 2157 4851 40  0001 C CNN
 F 2 "Resistors_ThroughHole:Resistor_Horizontal_RM10mm" V 2080 4850 30  0001 C CNN
 F 3 "~" H 2150 4850 30  0000 C CNN
@@
 F 3 "" H 900 1450 60  0000 C CNN
 	1    900  1450
-	-1   0    0    -1
+	-1   0    0    1
 $EndComp
 $Comp
@@
 L CONN_3 P3
 U 1 1 5787FAE3
-P 900 3950
-F 0 "P3" V 850 3950 50  0000 C CNN
-F 1 "CONN_3" V 950 3950 40  0000 C CNN
-F 2 "Connect:bornier3" H 900 3950 60  0001 C CNN
-F 3 "" H 900 3950 60  0000 C CNN
-	1    900  3950
+P 1200 3950
+F 0 "P3" V 1150 3950 50  0000 C CNN
+F 1 "CONN_3" V 1250 3950 40  0000 C CNN
+F 2 "Connect:bornier3" H 1200 3950 60  0001 C CNN
+F 3 "" H 1200 3950 60  0000 C CNN
+	1    1200 3950
 	-1   0    0    -1
 $EndComp
@@
 	1    0    0    -1
 $EndComp
-$Comp
-L FUSE F1
-U 1 1 5788B086
-P 1750 750
-F 0 "F1" H 1850 800 40  0000 C CNN
-F 1 "FUSE" H 1650 700 40  0000 C CNN
-F 2 "Fuse_Holders_and_Fuses:Fuseholder5x20_horiz_open_Schurter_0031_8201" H 1750 750 60  0001 C CNN
-F 3 "~" H 1750 750 60  0000 C CNN
-	1    1750 750
-	-1   0    0    1
-$EndComp
-Wire Wire Line
-	1250 750  1500 750
-Wire Wire Line
-	2000 750  2300 750
+Wire Wire Line
+	1250 750  2300 750
 Wire Wire Line
 	1250 1550 2300 1550
-Wire Wire Line
-	1500 750  1500 1350
-Wire Wire Line
-	1500 1350 1250 1350
-Wire Wire Line
-	1250 950  1400 950
-Wire Wire Line
-	1400 950  1400 1550
-Connection ~ 1400 1550
 $Comp
 L GND #PWR05
@@
 F 3 "" H 7000 1150 60  0000 C CNN
 	1    7000 1150
-	-1   0    0    -1
+	-1   0    0    1
 $EndComp
 $Comp
@@
 $EndComp
 $Comp
-L FUSE F3
-U 1 1 5788C45D
-P 7700 1050
-F 0 "F3" H 7800 1100 40  0000 C CNN
-F 1 "FUSE" H 7600 1000 40  0000 C CNN
-F 2 "Fuse_Holders_and_Fuses:Fuseholder5x20_horiz_open_Schurter_0031_8201" H 7700 1050 60  0001 C CNN
-F 3 "~" H 7700 1050 60  0000 C CNN
-	1    7700 1050
-	-1   0    0    1
-$EndComp
-$Comp
 L GND #PWR06
 U 1 1 5788C46B
@@
 L JUMPER3 JP1
 U 1 1 578E85FB
-P 6900 4550
-F 0 "JP1" H 6950 4450 50  0000 L CNN
-F 1 "JUMPER3" H 6900 4650 50  0000 C BNN
-F 2 "Pin_Headers:Pin_Header_Straight_1x03" H 6900 4550 50  0001 C CNN
-F 3 "" H 6900 4550 50  0000 C CNN
-	1    6900 4550
-	-1   0    0    -1
+P 6900 4850
+F 0 "JP1" H 6950 4750 50  0000 L CNN
+F 1 "JUMPER3" H 6900 4950 50  0000 C BNN
+F 2 "Pin_Headers:Pin_Header_Straight_1x03" H 6900 4850 50  0001 C CNN
+F 3 "" H 6900 4850 50  0000 C CNN
+	1    6900 4850
+	-1   0    0    1
 $EndComp
 Wire Wire Line
@@
 	1    0    0    -1
 $EndComp
-$Comp
-L FUSE F2
-U 1 1 578EBA34
-P 4700 750
-F 0 "F2" H 4800 800 40  0000 C CNN
-F 1 "FUSE" H 4600 700 40  0000 C CNN
-F 2 "Fuse_Holders_and_Fuses:Fuseholder5x20_horiz_open_Schurter_0031_8201" H 4700 750 60  0001 C CNN
-F 3 "~" H 4700 750 60  0000 C CNN
-	1    4700 750
-	-1   0    0    1
-$EndComp
-Wire Wire Line
-	4200 750  4450 750
-Wire Wire Line
-	4950 750  6100 750
+Wire Wire Line
+	4200 750  6100 750
 Wire Wire Line
 	4200 950  4350 950
@@
 F 0 "C4" H 6275 850 50  0000 L CNN
 F 1 "100n" H 6275 650 50  0000 L CNN
-F 2 "Capacitors_ThroughHole:C_Rect_L7_W2_P5" H 6288 600 50  0001 C CNN
+F 2 "Capacitors_ThroughHole:C_Rect_L18_W6_H12_P15" H 6288 600 50  0001 C CNN
 F 3 "" H 6250 750 50  0000 C CNN
 	1    6250 750
@@
 Text Label 4200 6000 0    60   ~ 0
 IA
-Text Label 7300 4550 2    60   ~ 0
+Text Label 7300 4850 2    60   ~ 0
 UA
-Text Label 6300 4550 0    60   ~ 0
+Text Label 6300 4850 0    60   ~ 0
 CS_ADC
 Wire Wire Line
-	7300 4550 7150 4550
-Wire Wire Line
-	6650 4550 6300 4550
+	7300 4850 7150 4850
+Wire Wire Line
+	6650 4850 6300 4850
 $Comp
 L JUMPER3 JP2
 U 1 1 578F703D
-P 6900 4850
-F 0 "JP2" H 6950 4750 50  0000 L CNN
-F 1 "JUMPER3" H 6900 4950 50  0000 C BNN
-F 2 "Pin_Headers:Pin_Header_Straight_1x03" H 6900 4850 50  0001 C CNN
-F 3 "" H 6900 4850 50  0000 C CNN
-	1    6900 4850
-	-1   0    0    1
-$EndComp
-Wire Wire Line
-	7300 4850 7150 4850
-Wire Wire Line
-	6650 4850 6300 4850
-Text Label 6300 4850 0    60   ~ 0
+P 6900 4550
+F 0 "JP2" H 6950 4450 50  0000 L CNN
+F 1 "JUMPER3" H 6900 4650 50  0000 C BNN
+F 2 "Pin_Headers:Pin_Header_Straight_1x03" H 6900 4550 50  0001 C CNN
+F 3 "" H 6900 4550 50  0000 C CNN
+	1    6900 4550
+	-1   0    0    -1
+$EndComp
+Wire Wire Line
+	7300 4550 7150 4550
+Wire Wire Line
+	6650 4550 6300 4550
+Text Label 6300 4550 0    60   ~ 0
 CS_DAC
-Text Label 7300 4850 2    60   ~ 0
+Text Label 7300 4550 2    60   ~ 0
 IA
 Wire Wire Line
@@
 Wire Wire Line
 	10300 3850 9900 3850
-Text Label 1500 3950 2    60   ~ 0
+Text Label 1800 3950 2    60   ~ 0
 UK
 Wire Wire Line
-	1250 4050 1500 4050
-Wire Wire Line
-	1500 3950 1250 3950
+	1550 4050 2350 4050
+Wire Wire Line
+	1800 3950 1550 3950
 Text Label 4200 6400 0    60   ~ 0
 UA
@@
 Wire Wire Line
 	2750 3700 2750 3750
-Wire Wire Line
-	2350 4050 2350 4850
-Wire Wire Line
-	2350 4050 2000 4050
 Connection ~ 2150 4050
 Text Label 1850 4600 0    60   ~ 0
 UG
-Text Label 1500 4050 2    60   ~ 0
+Text Label 1800 4050 2    60   ~ 0
 GRID
 $Comp
 L A+ #PWR025
 U 1 1 578FD605
-P 1250 3750
-F 0 "#PWR025" H 1250 3700 20  0001 C CNN
-F 1 "A+" H 1250 3850 30  0000 C CNN
-F 2 "" H 1250 3750 60  0000 C CNN
-F 3 "" H 1250 3750 60  0000 C CNN
-	1    1250 3750
-	1    0    0    -1
-$EndComp
-Wire Wire Line
-	1250 3750 1250 3850
+P 1550 3750
+F 0 "#PWR025" H 1550 3700 20  0001 C CNN
+F 1 "A+" H 1550 3850 30  0000 C CNN
+F 2 "" H 1550 3750 60  0000 C CNN
+F 3 "" H 1550 3750 60  0000 C CNN
+	1    1550 3750
+	1    0    0    -1
+$EndComp
+Wire Wire Line
+	1550 3750 1550 3850
 Wire Wire Line
 	4650 3050 4650 3250
@@
 F 0 "C5" H 6275 1650 50  0000 L CNN
 F 1 "100n" H 6275 1450 50  0000 L CNN
-F 2 "Capacitors_ThroughHole:C_Rect_L7_W2_P5" H 6288 1400 50  0001 C CNN
+F 2 "Capacitors_ThroughHole:C_Rect_L18_W6_H12_P15" H 6288 1400 50  0001 C CNN
 F 3 "" H 6250 1550 50  0000 C CNN
 	1    6250 1550
@@
 Connection ~ 5250 1550
 Wire Wire Line
-	7350 1050 7450 1050
-Wire Wire Line
-	7950 750  7950 1050
+	7350 1050 7950 1050
+Wire Wire Line
+	7950 1050 7950 750
 Connection ~ 6500 750
 Wire Wire Line
@@
 P 2150 4300
 F 0 "R2" V 2150 4300 40  0000 C CNN
-F 1 "R" V 2157 4301 40  0001 C CNN
+F 1 "R2" V 2157 4301 40  0001 C CNN
 F 2 "Resistors_ThroughHole:Resistor_Horizontal_RM10mm" V 2080 4300 30  0001 C CNN
 F 3 "~" H 2150 4300 30  0000 C CNN
@@
 Wire Wire Line
 	3500 5650 3650 5650
-$Comp
-L C C9
-U 1 1 57908FFE
-P 3000 3700
-F 0 "C9" H 3025 3800 50  0000 L CNN
-F 1 "100n" H 3025 3600 50  0000 L CNN
-F 2 "Capacitors_ThroughHole:C_Rect_L7_W2_P5" H 3038 3550 50  0001 C CNN
-F 3 "" H 3000 3700 50  0000 C CNN
-	1    3000 3700
-	0    1    -1   0
-$EndComp
-Connection ~ 3150 3950
-Wire Wire Line
-	2850 3700 2750 3700
-$Comp
-L C C8
-U 1 1 57909443
-P 2950 4500
-F 0 "C8" H 2975 4600 50  0000 L CNN
-F 1 "100n" H 2975 4400 50  0000 L CNN
-F 2 "Capacitors_ThroughHole:C_Rect_L7_W2_P5" H 2988 4350 50  0001 C CNN
-F 3 "" H 2950 4500 50  0000 C CNN
-	1    2950 4500
-	-1   0    0    -1
-$EndComp
-Wire Wire Line
-	2750 4350 2950 4350
-$Comp
-L GND #PWR031
-U 1 1 5790991C
-P 2950 4700
-F 0 "#PWR031" H 2950 4700 30  0001 C CNN
-F 1 "GND" H 2950 4630 30  0001 C CNN
-F 2 "" H 2950 4700 60  0000 C CNN
-F 3 "" H 2950 4700 60  0000 C CNN
-	1    2950 4700
-	1    0    0    -1
-$EndComp
-Wire Wire Line
-	2950 4650 2950 4700
-Wire Wire Line
-	2350 4850 2550 4850
-Wire Wire Line
-	3050 4850 3200 4850
-Wire Wire Line
-	3200 4850 3200 4150
+Wire Wire Line
+	2350 4650 2550 4650
+Wire Wire Line
+	3050 4650 3200 4650
 Wire Wire Line
 	4950 4050 4950 4250
@@
 	4150 4450 4350 4450
 $Comp
-L GND #PWR032
+L GND #PWR031
 U 1 1 5790A4B3
 P 4350 4800
-F 0 "#PWR032" H 4350 4800 30  0001 C CNN
+F 0 "#PWR031" H 4350 4800 30  0001 C CNN
 F 1 "GND" H 4350 4730 30  0001 C CNN
 F 2 "" H 4350 4800 60  0000 C CNN
@@
 $EndComp
 $Comp
-L GND #PWR033
+L GND #PWR032
 U 1 1 5790C62B
 P 3700 6650
-F 0 "#PWR033" H 3700 6650 30  0001 C CNN
+F 0 "#PWR032" H 3700 6650 30  0001 C CNN
 F 1 "GND" H 3700 6580 30  0001 C CNN
 F 2 "" H 3700 6650 60  0000 C CNN
@@
 	4850 5650 4850 5700
 $Comp
-L GND #PWR034
+L GND #PWR033
 U 1 1 57910308
 P 10400 4900
-F 0 "#PWR034" H 10400 4900 30  0001 C CNN
+F 0 "#PWR033" H 10400 4900 30  0001 C CNN
 F 1 "GND" H 10400 4830 30  0001 C CNN
 F 2 "" H 10400 4900 60  0000 C CNN
@@
 $EndComp
 $Comp
-L VDD #PWR035
+L VDD #PWR034
 U 1 1 579103AF
 P 10250 5000
-F 0 "#PWR035" H 10250 5100 30  0001 C CNN
+F 0 "#PWR034" H 10250 5100 30  0001 C CNN
 F 1 "VDD" H 10250 5110 30  0000 C CNN
 F 2 "" H 10250 5000 60  0000 C CNN
@@
 Text Label 10300 4750 2    60   ~ 0
 LCD_RS
+Wire Wire Line
+	3150 3950 3150 4000
+Wire Wire Line
+	2350 4050 2350 4650
+Wire Wire Line
+	3200 4650 3200 4150
+Wire Wire Line
+	1250 950  1250 1350
+Wire Wire Line
+	1450 1550 1450 750
+Connection ~ 1450 750
+Connection ~ 1450 1550
 $EndSCHEMATC

Commit message: Fix diode bridges footprints in PCB
Connections:
- net at D1.2, P1.1 (P1), P2.1 (P1): no longer D1.4
- net at P1.2 (PM), P2.2 (PM): now also D1.4
Changed lines of the file:
@@
 U 1 1 5788A706
 P 2300 1150
-F 0 "D1" H 2050 1450 50  0000 C CNN
-F 1 "B80C1500" H 2550 800 50  0000 C CNN
+F 0 "D1" H 2050 850 50  0000 C CNN
+F 1 "B80C1500" H 2550 1500 50  0000 C CNN
 F 2 "w_pth_diodes:bridge_wob" H 2300 1150 50  0001 C CNN
 F 3 "" H 2300 1150 50  0000 C CNN
 	1    2300 1150
-	1    0    0    -1
+	1    0    0    1
 $EndComp
 $Comp
@@
 Wire Wire Line
 	1250 750  2300 750
-Wire Wire Line
-	1250 1550 2300 1550
 $Comp
 L GND #PWR05
@@
 	1250 950  1250 1350
 Wire Wire Line
+	1250 1550 1450 1550
+Wire Wire Line
 	1450 1550 1450 750
 Connection ~ 1450 750
-Connection ~ 1450 1550
+Wire Wire Line
+	1250 1350 1750 1350
+Wire Wire Line
+	1750 1350 1750 1550
+Wire Wire Line
+	1750 1550 2300 1550
 $EndSCHEMATC

Commit message: Optimize routing & silkscreen
Parts:
- removed C12: 100n, Capacitors_ThroughHole:C_Rect_L7_W2_P5, symbol C
- added JP3: JUMPER, freetronics_footprints:SJ_OPEN, symbol JUMPER
- P3: value CONN_3 -> TO_TUBE
Connections:
- net DAC_OUT: now also JP3.1; no longer SHIELD1.AD0
- net GND: now also SHIELD1.GND3
- new net: JP3.2, SHIELD1.AD0
- no-connect marks 18 -> 17
Changed lines of the file:
@@
 P 1200 3950
 F 0 "P3" V 1150 3950 50  0000 C CNN
-F 1 "CONN_3" V 1250 3950 40  0000 C CNN
+F 1 "TO_TUBE" V 1250 3950 40  0000 C CNN
 F 2 "Connect:bornier3" H 1200 3950 60  0001 C CNN
 F 3 "" H 1200 3950 60  0000 C CNN
@@
 Wire Wire Line
 	8000 4250 7550 4250
-Text Label 7550 4450 0    60   ~ 0
+Text Label 6200 4250 0    60   ~ 0
 DAC_OUT
 Text Label 7550 4550 0    60   ~ 0
@@
 	7550 4550 8000 4550
 Wire Wire Line
-	8000 4450 7550 4450
+	7450 4450 8000 4450
 Text Label 10300 4450 2    60   ~ 0
 LCD_D5
@@
 	4150 4500 4150 4450
 Wire Wire Line
-	4150 3650 4150 3850
-Wire Wire Line
 	3750 2650 3750 4900
 Wire Wire Line
@@
 	4650 3050 4650 3250
 Wire Wire Line
-	4650 3250 5850 3250
-Wire Wire Line
 	5850 3250 5850 2250
-Wire Wire Line
-	4850 2250 6000 2250
 Text Label 5900 4050 2    60   ~ 0
 PWM_OUT
@@
 Wire Notes Line
 	4150 2000 4150 3300
-Wire Notes Line
-	4150 2000 6250 2000
-Text Notes 6250 3400 2    60   ~ 0
+Text Notes 6000 3400 2    60   ~ 0
 OPTIONAL
 Wire Notes Line
@@
 	10100 1750 10100 1900
 $Comp
-L C C12
-U 1 1 579081F5
-P 6000 2600
-F 0 "C12" H 6025 2700 50  0000 L CNN
-F 1 "100n" H 6025 2500 50  0000 L CNN
-F 2 "Capacitors_ThroughHole:C_Rect_L7_W2_P5" H 6038 2450 50  0001 C CNN
-F 3 "" H 6000 2600 50  0000 C CNN
-	1    6000 2600
-	1    0    0    1
-$EndComp
-Wire Notes Line
-	6250 2000 6250 3300
-$Comp
-L GND #PWR028
-U 1 1 57908535
-P 6000 2800
-F 0 "#PWR028" H 6000 2800 30  0001 C CNN
-F 1 "GND" H 6000 2730 30  0001 C CNN
-F 2 "" H 6000 2800 60  0000 C CNN
-F 3 "" H 6000 2800 60  0000 C CNN
-	1    6000 2800
-	1    0    0    -1
-$EndComp
-Wire Wire Line
-	6000 2250 6000 2450
-Connection ~ 5850 2250
-Wire Wire Line
-	6000 2750 6000 2800
-$Comp
 L C C15
 U 1 1 57908847
@@
 $EndComp
 $Comp
-L GND #PWR029
+L GND #PWR028
 U 1 1 57908946
 P 5750 5750
-F 0 "#PWR029" H 5750 5750 30  0001 C CNN
+F 0 "#PWR028" H 5750 5750 30  0001 C CNN
 F 1 "GND" H 5750 5680 30  0001 C CNN
 F 2 "" H 5750 5750 60  0000 C CNN
@@
 $EndComp
 $Comp
-L GND #PWR030
+L GND #PWR029
 U 1 1 57908CF6
 P 3950 5700
-F 0 "#PWR030" H 3950 5700 30  0001 C CNN
+F 0 "#PWR029" H 3950 5700 30  0001 C CNN
 F 1 "GND" H 3950 5630 30  0001 C CNN
 F 2 "" H 3950 5700 60  0000 C CNN
@@
 	4150 4450 4350 4450
 $Comp
-L GND #PWR031
+L GND #PWR030
 U 1 1 5790A4B3
 P 4350 4800
-F 0 "#PWR031" H 4350 4800 30  0001 C CNN
+F 0 "#PWR030" H 4350 4800 30  0001 C CNN
 F 1 "GND" H 4350 4730 30  0001 C CNN
 F 2 "" H 4350 4800 60  0000 C CNN
@@
 Wire Notes Line
 	3800 4950 6000 4950
-Wire Notes Line
-	6250 3300 4150 3300
 $Comp
 L C C13
@@
 $EndComp
 $Comp
-L GND #PWR032
+L GND #PWR031
 U 1 1 5790C62B
 P 3700 6650
-F 0 "#PWR032" H 3700 6650 30  0001 C CNN
+F 0 "#PWR031" H 3700 6650 30  0001 C CNN
 F 1 "GND" H 3700 6580 30  0001 C CNN
 F 2 "" H 3700 6650 60  0000 C CNN
@@
 	4850 5650 4850 5700
 $Comp
-L GND #PWR033
+L GND #PWR032
 U 1 1 57910308
-P 10400 4900
-F 0 "#PWR033" H 10400 4900 30  0001 C CNN
-F 1 "GND" H 10400 4830 30  0001 C CNN
-F 2 "" H 10400 4900 60  0000 C CNN
-F 3 "" H 10400 4900 60  0000 C CNN
-	1    10400 4900
-	-1   0    0    -1
-$EndComp
-$Comp
-L VDD #PWR034
+P 10400 4875
+F 0 "#PWR032" H 10400 4875 30  0001 C CNN
+F 1 "GND" H 10400 4805 30  0001 C CNN
+F 2 "" H 10400 4875 60  0000 C CNN
+F 3 "" H 10400 4875 60  0000 C CNN
+	1    10400 4875
+	-1   0    0    -1
+$EndComp
+$Comp
+L VDD #PWR033
 U 1 1 579103AF
-P 10250 5000
-F 0 "#PWR034" H 10250 5100 30  0001 C CNN
-F 1 "VDD" H 10250 5110 30  0000 C CNN
-F 2 "" H 10250 5000 60  0000 C CNN
-F 3 "" H 10250 5000 60  0000 C CNN
-	1    10250 5000
+P 10250 4950
+F 0 "#PWR033" H 10250 5050 30  0001 C CNN
+F 1 "VDD" H 10250 5060 30  0000 C CNN
+F 2 "" H 10250 4950 60  0000 C CNN
+F 3 "" H 10250 4950 60  0000 C CNN
+	1    10250 4950
 	-1   0    0    -1
 $EndComp
@@
 Wire Notes Line
 	4300 5400 6050 5400
-NoConn ~ 9900 3450
 NoConn ~ 9900 3350
 NoConn ~ 9900 4050
@@
 	10500 3150 9900 3150
 Wire Wire Line
-	10400 4850 10400 4900
-Wire Wire Line
 	10400 4850 10550 4850
 Wire Wire Line
-	10550 4950 10500 4950
-Wire Wire Line
-	10500 4950 10500 5000
-Wire Wire Line
-	10500 5000 10250 5000
+	10250 4950 10550 4950
 Text Label 10300 3150 2    60   ~ 0
 SCL
@@
 Wire Wire Line
 	1750 1550 2300 1550
+$Comp
+L GND #PWR034
+U 1 1 5794FAD8
+P 10000 3475
+F 0 "#PWR034" H 10000 3475 30  0001 C CNN
+F 1 "GND" H 10000 3405 30  0001 C CNN
+F 2 "" H 10000 3475 60  0000 C CNN
+F 3 "" H 10000 3475 60  0000 C CNN
+	1    10000 3475
+	-1   0    0    -1
+$EndComp
+Wire Wire Line
+	9900 3450 10000 3450
+Wire Wire Line
+	10000 3450 10000 3475
+Wire Wire Line
+	10400 4875 10400 4850
+Wire Wire Line
+	5850 2250 4850 2250
+Wire Wire Line
+	4150 3650 4150 3850
+Wire Wire Line
+	4650 3250 5850 3250
+Wire Notes Line
+	6000 2000 6000 3300
+Wire Notes Line
+	4150 2000 6000 2000
+Wire Notes Line
+	6000 3300 4150 3300
+$Comp
+L JUMPER JP3
+U 1 1 579801B2
+P 6900 4250
+F 0 "JP3" H 6900 4400 50  0000 C CNN
+F 1 "JUMPER" H 6900 4170 50  0000 C CNN
+F 2 "freetronics_footprints:SJ_OPEN" H 6900 4250 50  0001 C CNN
+F 3 "" H 6900 4250 50  0000 C CNN
+	1    6900 4250
+	1    0    0    -1
+$EndComp
+Wire Wire Line
+	6200 4250 6600 4250
+Wire Wire Line
+	7200 4250 7450 4250
+Wire Wire Line
+	7450 4250 7450 4450
 $EndSCHEMATC
