File: kicad/nanoTracer.sch (KiCad schematic (older format))
At the start: 45 parts, among them J1 SIL10, P1 6.3_AC, P2 HEATER, P3 TO_TUBE, P4 HT_AC, P5 NEG_AC, U1 TL072, U2 TL071, U3 MCP4921-E/P, U4 LM337T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

Commit message: Added headers for unconnected Arduino pins
Parts:
- added P6, P7: CONN_2, Pin_Headers:Pin_Header_Straight_1x02, symbol CONN_2
Connections:
- net D8: now reaches SHIELD1.8
- net D8: now also P7.2 (P2)
- net D9: now reaches SHIELD1.9
- net D9: now also P7.1 (P1)
- net at SHIELD1.AD4: now also P6.1 (P1)
- net at SHIELD1.AD5: now also P6.2 (P2)
- no-connect marks 17 -> 13
Changed lines of the file:
@@
 	-1   0    0    -1
-$EndComp
-NoConn ~ 8000 4850
-$Comp
-L ARDUINO_SHIELD SHIELD1
-U 1 1 578EA1FF
-P 8950 4150
-F 0 "SHIELD1" H 8500 5300 60  0000 C CNN
-F 1 "ARDUINO_SHIELD" H 9000 3200 60  0000 C CNN
-F 2 "freetronics_footprints:ARDUINO_SHIELD" H 8950 3950 50  0001 C CNN
-F 3 "" H 8950 4150 60  0000 C CNN
-	1    8950 4150
-	1    0    0    -1
 $EndComp
 NoConn ~ 9900 4850
 NoConn ~ 9900 4950
-NoConn ~ 9900 3950
 NoConn ~ 8000 3950
 NoConn ~ 8000 3750
@@
 	4300 5400 6050 5400
 NoConn ~ 9900 3350
-NoConn ~ 9900 4050
-NoConn ~ 8000 4950
 $Comp
 L SIL10 J1
@@
 Wire Wire Line
 	7450 4250 7450 4450
+$Comp
+L ARDUINO_SHIELD SHIELD1
+U 1 1 578EA1FF
+P 8950 4150
+F 0 "SHIELD1" H 8500 5300 60  0000 C CNN
+F 1 "ARDUINO_SHIELD" H 9000 3200 60  0000 C CNN
+F 2 "freetronics_footprints:ARDUINO_SHIELD" H 8950 3950 50  0001 C CNN
+F 3 "" H 8950 4150 60  0000 C CNN
+	1    8950 4150
+	1    0    0    -1
+$EndComp
+$Comp
+L CONN_2 P6
+U 1 1 579F98D5
+P 7325 5225
+F 0 "P6" V 7275 5225 40  0000 C CNN
+F 1 "CONN_2" V 7375 5225 40  0000 C CNN
+F 2 "Pin_Headers:Pin_Header_Straight_1x02" H 7325 5225 60  0001 C CNN
+F 3 "" H 7325 5225 60  0000 C CNN
+	1    7325 5225
+	-1   0    0    -1
+$EndComp
+Wire Wire Line
+	7775 5125 7775 4850
+Wire Wire Line
+	7775 4850 8000 4850
+Wire Wire Line
+	7675 5325 7875 5325
+Wire Wire Line
+	7875 5325 7875 4950
+Wire Wire Line
+	7875 4950 8000 4950
+Wire Wire Line
+	7675 5125 7775 5125
+$Comp
+L CONN_2 P7
+U 1 1 579FAA3F
+P 10825 2750
+F 0 "P7" V 10775 2750 40  0000 C CNN
+F 1 "CONN_2" V 10875 2750 40  0000 C CNN
+F 2 "Pin_Headers:Pin_Header_Straight_1x02" H 10825 2750 60  0001 C CNN
+F 3 "" H 10825 2750 60  0000 C CNN
+	1    10825 2750
+	1    0    0    -1
+$EndComp
+Text Label 10300 3950 2    60   ~ 0
+D9
+Text Label 10300 4050 2    60   ~ 0
+D8
+Wire Wire Line
+	9900 3950 10300 3950
+Wire Wire Line
+	9900 4050 10300 4050
+Text Label 10300 2650 0    60   ~ 0
+D9
+Text Label 10300 2850 0    60   ~ 0
+D8
+Wire Wire Line
+	10300 2850 10475 2850
+Wire Wire Line
+	10300 2650 10475 2650
 $EndSCHEMATC
